Commit message: 添加了一个启动文件start_navigation，用于发起定点导航

File: src/mybot_description/urdf/mybot.xacro (robot description, xacro)
@@ -190,3 +190,29 @@
     </inertial>
   </link>
+  <!-- Localization model -->
+  <joint name="localization_joint" type="fixed">
+    <axis xyz="0 1 0" />
+    <origin xyz=".05 0 .1" rpy="0 0 0"/>
+    <parent link="chassis"/>
+    <child link="Localization"/>
+  </joint>
+  <link name="Localization">
+    <collision>
+      <origin xyz="0 0 0" rpy="0 0 0"/>
+      <geometry>
+        <box size="0.05 0.05 0.05"/>
+      </geometry>
+    </collision>
+    <visual>
+      <origin xyz="0 0 0" rpy="0 0 0"/>
+      <geometry>
+        <box size="0.05 0.05 0.05"/>
+      </geometry>
+    </visual>
+    <inertial>
+      <mass value="1e-5" />
+      <origin xyz="0 0 0" rpy="0 0 0"/>
+      <inertia ixx="1e-6" ixy="0" ixz="0" iyy="1e-6" iyz="0" izz="1e-6" />
+    </inertial>
+  </link>
 </robot>
